Commit message: Initial commit. Some adjustments from base repo already made.

File: urdf/03-origins.urdf (robot description, URDF)
Before this commit: robot origins, 2 links, 1 joints
Links:
- added link left_leg; visual box size=0.6 0.1 0.2
Joints:
- added joint base_to_left_leg: type fixed, parent base_link, child left_leg, origin xyz=0.0 0.22 0.25 rpy=0.0 -0.8 0.0

File: urdf/04-materials.urdf (robot description, URDF)
Before this commit: robot materials, 3 links, 2 joints
Links:
- added link right_wheel; visual cylinder length=0.08 radius=0.06
Joints:
- added joint right_leg_to_right_wheel: type revolute, parent right_leg, child right_wheel, origin xyz=0 0 -0.6 rpy=0 0 0, axis 0 1 0, limit lower=-1.57 upper=1.57 effort=10.0 velocity=1.0
