Commit message: Added some dimensions to tail. Cheetah body does not have reasonable dimensions yet.

File: urdf/box_tail.urdf (robot description, URDF)
Before this commit: robot box_with_rod, 3 links, 2 joints
Links:
- link box: mass None -> 50.0; geometry collision box size=1.3 0.4 0.4; visual box size=1.3 0.4 0.4
- link rod: mass None -> 2.0; geometry collision cylinder length=0.7 radius=0.05; visual cylinder length=0.7 radius=0.05
Joints:
- joint box_to_rod: limit lower=-1.57 upper=1.57 effort=10.0 velocity=1.0 -> (none); type revolute -> continuous

Commit message: Added endeffector

File: urdf/box_tail.urdf (robot description, URDF)
Before this commit: robot box_with_rod, 3 links, 2 joints
Links:
- added link endeffector
Joints:
- added joint rod_to_endeffector: type fixed, parent rod, child endeffector, origin xyz=0 0 0.7 rpy=0 0 0
